Commit message: Fixed Warning: 'Joint state with name: left_wheel_joint was received but not found in URDF'

File: create_description/urdf/create_xl.urdf.xacro (robot description, xacro)
@@ -13,3 +13,29 @@
     </visual>
   </link>
+  <link name="left_wheel_link">
+    <inertial>
+    <origin xyz="0 0 0" />
+    <mass value="0.01" />
+    <inertia ixx="0.001" ixy="0.0" ixz="0.0" iyy="0.001" iyz="0.0" izz="0.001" />
+    </inertial>
+  </link>
+  <joint name="left_wheel_joint" type="continuous">
+    <origin xyz="0 0.1175 0.015" rpy="0 0 0" />
+    <parent link="base_link" />
+    <child link="left_wheel_link" />
+    <axis xyz="0 1 0" />
+  </joint>
+  <link name="right_wheel_link">
+    <inertial>
+    <origin xyz="0 0 0" />
+    <mass value="0.01" />
+    <inertia ixx="0.001" ixy="0.0" ixz="0.0" iyy="0.001" iyz="0.0" izz="0.001" />
+    </inertial>
+  </link>
+  <joint name="right_wheel_joint" type="continuous">
+    <origin xyz="0 0.1175 0.015" rpy="0 0 0" />
+    <parent link="base_link" />
+    <child link="right_wheel_link" />
+    <axis xyz="0 1 0" />
+  </joint>
 </robot>

Commit message: Navigation Package. Not working yet

File: create_description/urdf/create_xl.urdf.xacro (robot description, xacro)
@@ -34,5 +34,5 @@
   </link>
   <joint name="right_wheel_joint" type="continuous">
-    <origin xyz="0 0.1175 0.015" rpy="0 0 0" />
+    <origin xyz="0 -0.1175 0.015" rpy="0 0 0" />
     <parent link="base_link" />
     <child link="right_wheel_link" />

Commit message: Fixed 3D model and cameras tranformations. Fixed bug with 'create_fix'odom.py' bug.

File: create_description/urdf/create_xl.urdf.xacro (robot description, xacro)
@@ -1,21 +1,21 @@
 <?xml version="1.0" ?>
 <robot name="create_2" xmlns:xacro="http://ros.org/wiki/xacro">
-  <material name="Orange">
+  <material name="Gray">
     <color rgba="${150/255} ${150/255} ${150/255} 1.0"/>
   </material>
   <link name="base_link">
     <visual>
-      <origin rpy="1.5708 0 1.5708" xyz="0 0 0.339"/>
+      <origin rpy="1.5708 0 1.5708" xyz="0 0 0.34315"/>
       <geometry>
         <mesh filename="package://create_description/meshes/create_xl.stl" scale="0.001 0.001 0.001"/>
       </geometry>
-      <material name="Orange"/>
+      <material name="Gray"/>
     </visual>
   </link>
   <link name="left_wheel_link">
     <inertial>
-    <origin xyz="0 0 0" />
-    <mass value="0.01" />
-    <inertia ixx="0.001" ixy="0.0" ixz="0.0" iyy="0.001" iyz="0.0" izz="0.001" />
+      <origin xyz="0 0 0" />
+      <mass value="0.01" />
+      <inertia ixx="0.001" ixy="0.0" ixz="0.0" iyy="0.001" iyz="0.0" izz="0.001" />
     </inertial>
   </link>
